Commit message: robot_sim -v1.2 -20210414

File: urdf/xacro/camera.urdf.xacro (robot description, xacro)
@@ -1,3 +1,4 @@
-<robot name="camera" xmlns:xacro="http://wiki.ros.org/xacro">
+<?xml version="1.0"?>
+<robot name="camera" xmlns:xacro="http://ros.org/wiki/xacro">
     <xacro:property name="camera_length" value="0.01" />
     <xacro:property name="camera_width" value="0.025" />
@@ -6,4 +7,5 @@
     <xacro:property name="camera_y" value="0.0" />
     <xacro:property name="camera_z" value="${base_link_length / 2 + camera_height / 2}" />
+    <xacro:property name="camera_m" value="0.01" />
     <link name="camera">
         <visual>
@@ -14,4 +16,11 @@
             <material name="black" />
         </visual>
+        <collision>
+            <geometry>
+                <box size="${camera_length} ${camera_width} ${camera_height}" />
+            </geometry>
+            <origin xyz="0.0 0.0 0.0" rpy="0.0 0.0 0.0" />
+        </collision>
+        <xacro:Box_inertial_matrix m="${camera_m}" l="${camera_length}" w="${camera_width}" h="${camera_height}" />
     </link>
     <joint name="camera2base_link" type="fixed">
@@ -20,3 +29,6 @@
         <origin xyz="${camera_x} ${camera_y} ${camera_z}" />
     </joint>
+    <gazebo reference="camera">
+        <material>Gazebo/Blue</material>
+    </gazebo>
 </robot>

File: urdf/xacro/car_base.urdf.xacro (robot description, xacro)
@@ -1,3 +1,4 @@
-<robot name="car_base" xmlns:xacro="http://www.ros.org/wiki/xacro">
+<?xml version="1.0"?>
+<robot name="car_base" xmlns:xacro="http://ros.org/wiki/xacro">
     <xacro:property name="PI" value="3.141"/>
     <material name="black">
@@ -8,4 +9,5 @@
     <xacro:property name="base_link_length" value="0.08" />
     <xacro:property name="earth_space" value="0.015" />
+    <xacro:property name="base_link_m" value="0.5" />
     <link name="base_footprint">
         <visual>
@@ -25,4 +27,11 @@
             </material>
         </visual>
+        <collision>
+            <geometry>
+                <cylinder radius="${base_link_radius}" length="${base_link_length}" />
+            </geometry>
+            <origin xyz="0 0 0" rpy="0 0 0" />
+        </collision>
+        <xacro:cylinder_inertial_matrix m="${base_link_m}" r="${base_link_radius}" h="${base_link_length}" />
     </link>
     <joint name="base_link2base_footprint" type="fixed">
@@ -31,6 +40,10 @@
         <origin xyz="0 0 ${earth_space + base_link_length / 2 }" />
     </joint>
+    <gazebo reference="base_link">
+        <material>Gazebo/Yellow</material>
+    </gazebo>
     <xacro:property name="wheel_radius" value="0.0325" />
     <xacro:property name="wheel_length" value="0.015" />
+    <xacro:property name="wheel_m" value="0.05" />
     <xacro:macro name="add_wheels" params="name flag">
         <link name="${name}_wheel">
@@ -42,4 +55,11 @@
                 <material name="black" />
             </visual>
+            <collision>
+                <geometry>
+                    <cylinder radius="${wheel_radius}" length="${wheel_length}" />
+                </geometry>
+                <origin xyz="0.0 0.0 0.0" rpy="${PI / 2} 0.0 0.0" />
+            </collision>
+            <xacro:cylinder_inertial_matrix m="${wheel_m}" r="${wheel_radius}" h="${wheel_length}"/>
         </link>
         <joint name="${name}_wheel2base_link" type="continuous">
@@ -49,10 +69,12 @@
             <axis xyz="0 1 0" />
         </joint>
+        <gazebo reference="${name}_wheel">
+            <material>Gazebo/Red</material>
+        </gazebo>
     </xacro:macro>
-    <xacro:add_wheels name="left" flag="1" />
-    <xacro:add_wheels name="right" flag="-1" />
     <xacro:property name="support_wheel_radius" value="0.0075" />
+    <xacro:property name="support_wheel_m" value="0.03" />
     <xacro:macro name="add_support_wheel" params="name flag" >
-        <link name="${name}_wheel">
+        <link name="${name}_support_wheel">
             <visual>
                 <geometry>
@@ -62,12 +84,24 @@
                 <material name="black" />
             </visual>
+            <collision>
+                <geometry>
+                    <sphere radius="${support_wheel_radius}" />
+                </geometry>
+                <origin xyz="0 0 0" rpy="0 0 0" />
+            </collision>
+            <xacro:sphere_inertial_matrix m="${support_wheel_m}" r="${support_wheel_radius}"/>
         </link>
         <joint name="${name}_wheel2base_link" type="continuous">
             <parent link="base_link" />
-            <child link="${name}_wheel" />
+            <child link="${name}_support_wheel" />
             <origin xyz="${flag * (base_link_radius - support_wheel_radius)} 0 ${-(base_link_length / 2 + earth_space / 2)}" />
             <axis xyz="1 1 1" />
         </joint>
+        <gazebo reference="${name}_support_wheel">
+            <material>Gazebo/Red</material>
+        </gazebo>
     </xacro:macro>
+    <xacro:add_wheels name="left" flag="1" />
+    <xacro:add_wheels name="right" flag="-1" />
     <xacro:add_support_wheel name="front" flag="1" />
     <xacro:add_support_wheel name="back" flag="-1" />

File: urdf/xacro/lidar.urdf.xacro (robot description, xacro)
@@ -1,3 +1,4 @@
-<robot name="my_laser" xmlns:xacro="http://wiki.ros.org/xacro">
+<?xml version="1.0"?>
+<robot name="lidar" xmlns:xacro="http://ros.org/wiki/xacro">
     <xacro:property name="support_length" value="0.15" />
     <xacro:property name="support_radius" value="0.01" />
@@ -5,4 +6,5 @@
     <xacro:property name="support_y" value="0.0" />
     <xacro:property name="support_z" value="${base_link_length / 2 + support_length / 2}" />
+    <xacro:property name="support_m" value="0.02" />
     <link name="support">
         <visual>
@@ -15,4 +17,11 @@
             </material>
         </visual>
+        <collision>
+            <geometry>
+                <cylinder radius="${support_radius}" length="${support_length}" />
+            </geometry>
+            <origin xyz="0.0 0.0 0.0" rpy="0.0 0.0 0.0" />
+        </collision>
+        <xacro:cylinder_inertial_matrix m="${support_m}" r="${support_radius}" h="${support_length}"/>
     </link>
     <joint name="support2base_link" type="fixed">
@@ -21,4 +30,7 @@
         <origin xyz="${support_x} ${support_y} ${support_z}" />
     </joint>
+    <gazebo reference="support">
+        <material>Gazebo/White</material>
+    </gazebo>
     <xacro:property name="laser_length" value="0.05" />
     <xacro:property name="laser_radius" value="0.03" />
@@ -26,4 +38,5 @@
     <xacro:property name="laser_y" value="0.0" />
     <xacro:property name="laser_z" value="${support_length / 2 + laser_length / 2}" />
+    <xacro:property name="laser_m" value="0.1" />
     <link name="laser">
         <visual>
@@ -34,4 +47,11 @@
             <material name="black" />
         </visual>
+        <collision>
+            <geometry>
+                <cylinder radius="${laser_radius}" length="${laser_length}" />
+            </geometry>
+            <origin xyz="0.0 0.0 0.0" rpy="0.0 0.0 0.0" />
+        </collision>
+        <xacro:cylinder_inertial_matrix m="${laser_m}" r="${laser_radius}" h="${laser_length}"/>
     </link>
     <joint name="laser2support" type="fixed">
@@ -40,3 +60,6 @@
         <origin xyz="${laser_x} ${laser_y} ${laser_z}" />
     </joint>
+    <gazebo reference="laser">
+        <material>Gazebo/Black</material>
+    </gazebo>
 </robot>

File: urdf/xacro/robot_car.urdf.xacro (robot description, xacro)
@@ -1,3 +1,5 @@
-<robot name="robot_car" xmlns:xacro="http://wiki.ros.org/xacro">
+<?xml version="1.0"?>
+<robot name="robot_car" xmlns:xacro="http://ros.org/wiki/xacro">
+    <xacro:include filename="inertial.urdf.xacro"/>
     <xacro:include filename="car_base.urdf.xacro"/>
     <xacro:include filename="lidar.urdf.xacro"/>

Commit message: robot_sim -v1.6 -20210419

File: urdf/xacro/camera.urdf.xacro (robot description, xacro)
@@ -15,5 +15,7 @@
             </geometry>
             <origin xyz="0.0 0.0 0.0" rpy="0.0 0.0 0.0" />
-            <material name="black" />
+            <material name="green"> <!-- easy to find front -->
+                <color rgba="0.0 1.0 0.0 1.0" />
+            </material>
         </visual>
         <collision>
@@ -31,5 +33,5 @@
     </joint>
     <gazebo reference="camera">
-        <material>Gazebo/Blue</material>
+        <material>Gazebo/Red</material>
     </gazebo>
 </robot>
